File: ttlclock3.kicad_pcb (KiCad board)
At the start: 2 copper layers, 149.9 x 99.1 mm, 71 parts, among them J1 USB power, J2 M, J3 M, SW1 Hold, SW2 Slow, SW3 Fast, U1 74LS14, U10 74LS74, U11 74LS74, U12 74LS74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

Commit message: Update to KiCad 7, not tested
Parts:
- J1: footprint Connectors:1X05 -> Connector_PinHeader_2.54mm:PinHeader_1x05_P2.54mm_Vertical
- J2, J3: footprint Connectors:1X01 -> Connector_PinHeader_2.54mm:PinHeader_1x01_P2.54mm_Vertical
- turned J1 to 0 degrees
Connections:
- net /H0/~Q0 renamed /H0/~{Q0}
- net /H0/~Q1 renamed /H0/~{Q1}
- net /H0/~R renamed /H0/~{R}
- net /H1/Ci renamed /H0/Co
- net /H1/~Q0 renamed /H1/~{Q0}
- net /H1/~Q1 renamed /H1/~{Q1}
- net /H2/Ci renamed /H1/Co
- net /H2/~Q0 renamed /H2/~{Q0}
- net /H2/~Q1 renamed /H2/~{Q1}
- net /M0/~Q0 renamed /M0/~{Q0}
- net /M0/~Q1 renamed /M0/~{Q1}
- net /M0/~R renamed /M0/~{R}
- net /M1/Ci renamed /M0/Co
- net /M1/~Q0 renamed /M1/~{Q0}
- net /M1/~Q1 renamed /M1/~{Q1}
- net /M2/Ci renamed /M1/Co
- net /M2/~Q0 renamed /M2/~{Q0}
- net /M2/~Q1 renamed /M2/~{Q1}
- net /M3/Ci renamed /M2/Co
- net /M3/~Q0 renamed /M3/~{Q0}
- net /M3/~Q1 renamed /M3/~{Q1}
- C24 pad 1: Net-(C24-Pad1) -> GND
- J1 pad 2: Net-(J1-Pad2) -> unconnected-(J1-Pin_2-Pad2)
- J1 pad 3: Net-(J1-Pad3) -> unconnected-(J1-Pin_3-Pad3)
- J1 pad 4: Net-(J1-Pad4) -> unconnected-(J1-Pin_4-Pad4)
- R24 pad 2: Net-(C24-Pad1) -> GND
- RN1 pad 9: Net-(RN1-Pad9) -> unconnected-(RN1-R8-Pad9)
- U16 pad 12: /H2/Co -> /H18
- U16 pad 5: /H18 -> /H2/Q1
- U2 pad 10: Net-(U2-Pad10) -> unconnected-(U2-I1c-Pad10)
- U2 pad 11: Net-(U2-Pad11) -> unconnected-(U2-I0c-Pad11)
- U2 pad 12: Net-(U2-Pad12) -> unconnected-(U2-Zd-Pad12)
- U2 pad 13: Net-(U2-Pad13) -> unconnected-(U2-I1d-Pad13)
- U2 pad 14: Net-(U2-Pad14) -> unconnected-(U2-I0d-Pad14)
- U2 pad 2: Net-(U2-Pad2) -> unconnected-(U2-I0a-Pad2)
- U2 pad 3: Net-(U2-Pad3) -> unconnected-(U2-I1a-Pad3)
- U2 pad 4: Net-(U2-Pad4) -> unconnected-(U2-Za-Pad4)
- U2 pad 9: Net-(U2-Pad9) -> unconnected-(U2-Zc-Pad9)
- U21 pad 1: /H2/Co -> /H18
- U21 pad 3: /H18 -> /H2/Q1
- U23 pad 13: Net-(U23-Pad13) -> unconnected-(U23A-Q-Pad13)
- U23 pad 5: Net-(U23-Pad5) -> unconnected-(U23B-Q-Pad5)
- U23 pad 7: Net-(C24-Pad1) -> GND
- U3 pad 12: Net-(U3-Pad12) -> unconnected-(U3-Zd-Pad12)
- U3 pad 13: Net-(U3-Pad13) -> unconnected-(U3-I1d-Pad13)
- U3 pad 14: Net-(U3-Pad14) -> unconnected-(U3-I0d-Pad14)
- U3 pad 2: Net-(U3-Pad2) -> unconnected-(U3-I0a-Pad2)
- U3 pad 3: Net-(U3-Pad3) -> unconnected-(U3-I1a-Pad3)
- U3 pad 4: Net-(U3-Pad4) -> unconnected-(U3-Za-Pad4)
- U3 pad 5: Net-(U3-Pad5) -> unconnected-(U3-I0b-Pad5)
- U3 pad 6: Net-(U3-Pad6) -> unconnected-(U3-I1b-Pad6)
- U3 pad 7: Net-(U3-Pad7) -> unconnected-(U3-Zb-Pad7)
- U4 pad 1: Net-(U4-Pad1) -> unconnected-(U4A-Q12-Pad1)
- U4 pad 13: Net-(U4-Pad13) -> unconnected-(U4A-Q9-Pad13)
- U4 pad 14: Net-(U4-Pad14) -> unconnected-(U4A-Q8-Pad14)
- U4 pad 15: Net-(U4-Pad15) -> unconnected-(U4A-Q10-Pad15)
- U4 pad 2: Net-(U4-Pad2) -> unconnected-(U4A-Q13-Pad2)
- U4 pad 4: Net-(U4-Pad4) -> unconnected-(U4A-Q6-Pad4)
- U4 pad 7: Net-(U4-Pad7) -> unconnected-(U4A-Q4-Pad7)
- U4 pad 9: Net-(U4-Pad9) -> unconnected-(U4A-P0-Pad9)
- U5 pad 10: Net-(U5-Pad10) -> unconnected-(U5B-Q1-Pad10)
- U5 pad 11: Net-(U5-Pad11) -> unconnected-(U5B-Q0-Pad11)
- U5 pad 5: Net-(U5-Pad5) -> unconnected-(U5A-Q2-Pad5)
Routing:
- net /H2/Q1: track 0.00 -> 28.2 mm, vias 0 -> 1
- net /M2/Co: track 46.8 -> 69.3 mm, vias 0 -> 1
- net /H1/Co: track 56.1 -> 77.7 mm
- net /M0/Co: track 40.8 -> 54.8 mm
- net Net-(C24-Pad1): track 12.4 -> 0.00 mm
- net /H0/~{R}: track 167.5 -> 155.2 mm
- net /H2/Co: track 12.4 -> 0.00 mm
- net /M1/Co: track 48.3 -> 60.1 mm, vias 0 -> 1
- net Net-(U4A-Q5): track 46.1 -> 36.8 mm
- net Net-(U13A-D): track 48.3 -> 57.5 mm
- net Net-(U11A-D): track 26.0 -> 33.8 mm
- net /H18: track 37.2 -> 44.9 mm
- net /H0/Co: track 41.7 -> 49.4 mm
- net +5V: track 720.0 -> 727.3 mm
- net /M54: track 88.7 -> 96.0 mm
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- added copper zone on F.Cu, net GND
- removed copper zone on F.Cu, net +5V
Other:
- net class Default removed
- net class POWER removed
